File: KICAD/CAN-Digital-Output-12V.kicad_pcb (KiCad board)
At the start: 2 copper layers, 84.1 x 75.4 mm, 46 parts, among them J1 UPDI Header, J2 Conn_01x04_Female, J3 UART Header, K1 CP1SA-12V-X, K2 CP1SA-12V-X, K3 CP1SA-12V-X, K4 CP1SA-12V-X, Q1 MMBT2222A-TP, Q2 MMBT2222A-TP, Q3 MMBT2222A-TP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

Commit message: Design review with Jarrod
Parts:
- removed D1, D2, D3, D4: NRVA4007T3G, Diode_SMD:D_SMA
- removed K1, K2, K3, K4: CP1SA-12V-X, eec:Panasonic-CP1SA-12V-X-MFG
- removed Q1, Q2, Q3, Q4: MMBT2222A-TP, Package_TO_SOT_SMD:SOT-23
- added J4: 0367831201, 0367831201:MOLEX_0367831201, F.Cu at (181.2, 101.9)
- U4, U6, U7, U8: value 1-2834011-3 -> VNL5050N3TR-E; footprint 1-2834011-3:CONN_1-2834011-3 -> Package_TO_SOT_SMD:SOT-223
- moved C1 58.3 mm to (152.1, 85.7)
- moved C2 58.3 mm to (161.8, 85.7)
- moved U1 58.3 mm to (157.0, 88.2)
- moved U8 55.3 mm to (168.9, 111.0), turned to 0 degrees
- moved U6 52.3 mm to (168.9, 103.4), turned to 0 degrees
- moved U7 50.2 mm to (168.9, 95.5), turned to 0 degrees
- moved U4 49.0 mm to (168.9, 87.1), turned to 0 degrees
- moved H4 47.3 mm to (157.0, 100.3)
- moved H2 47.3 mm to (154.2, 95.2)
- moved H3 47.3 mm to (152.1, 99.1)
- moved H1 47.3 mm to (158.8, 96.3)
- moved R8 35.8 mm to (171.8, 116.3)
- moved R10 34.7 mm to (171.8, 118.8)
- moved R9 34.2 mm to (171.7, 120.7)
- moved C5 28.7 mm to (130.3, 93.0)
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Connections:
- R10 pad 1: /RELAY_1 -> /OUT_4
- R10 pad 2: Net-(Q4-Pad1) -> Net-(R10-Pad2)
- R6 pad 1: /RELAY_1 -> /OUT_1
- R6 pad 2: Net-(Q1-Pad1) -> Net-(R6-Pad2)
- R8 pad 1: /RELAY_1 -> /OUT_2
- R8 pad 2: Net-(Q2-Pad1) -> Net-(R8-Pad2)
- R9 pad 1: /RELAY_1 -> /OUT_3
- R9 pad 2: Net-(Q3-Pad1) -> Net-(R9-Pad2)
- U3 pad 2: /RELAY_2 -> /OUT_2
- U3 pad 3: /RELAY_3 -> /OUT_3
- U3 pad 5: /RELAY_4 -> /OUT_4
- U3 pad 8: /RELAY_1 -> /OUT_1
- U4 pad 1: Net-(K1-Pad3) -> Net-(R6-Pad2)
- U4 pad 2: Net-(K1-Pad5) -> /DO_1
- U4 pad 3: Net-(K1-Pad4) -> GND
- U6 pad 1: Net-(K2-Pad3) -> Net-(R8-Pad2)
- U6 pad 2: Net-(K2-Pad5) -> /DO_2
- U6 pad 3: Net-(K2-Pad4) -> GND
- U7 pad 1: Net-(K3-Pad3) -> Net-(R9-Pad2)
- U7 pad 2: Net-(K3-Pad5) -> /DO_3
- U7 pad 3: Net-(K3-Pad4) -> GND
- U8 pad 1: Net-(K4-Pad3) -> Net-(R10-Pad2)
- U8 pad 2: Net-(K4-Pad5) -> /DO_4
- U8 pad 3: Net-(K4-Pad4) -> GND
Other:
- board size 84.1 x 75.4 mm -> 64.3 x 40.6 mm

Commit message: Third Design Review
Parts:
- removed H1, H2, H3, H4: MountingHole, MountingHole:MountingHole_2.2mm_M2_ISO14580
- removed J2: Conn_01x04_Female, Connector_PinHeader_1.27mm:PinHeader_1x04_P1.27mm_Vertical
- added D1: LED, LED_SMD:LED_0603_1608Metric_Pad1.05x0.95mm_HandSolder, F.Cu at (162.8, 86.4)
- added D2: LED, LED_SMD:LED_0603_1608Metric_Pad1.05x0.95mm_HandSolder, F.Cu at (162.8, 101.1)
- added D3: LED, LED_SMD:LED_0603_1608Metric_Pad1.05x0.95mm_HandSolder, F.Cu at (162.8, 93.7)
- added D4: LED, LED_SMD:LED_0603_1608Metric_Pad1.05x0.95mm_HandSolder, F.Cu at (162.8, 108.5)
- added R11: 150, Resistor_SMD:R_0603_1608Metric_Pad0.98x0.95mm_HandSolder, F.Cu at (162.8, 88.1)
- added R12: 150, Resistor_SMD:R_0603_1608Metric_Pad0.98x0.95mm_HandSolder, F.Cu at (162.8, 102.9)
- added R13: 150, Resistor_SMD:R_0603_1608Metric_Pad0.98x0.95mm_HandSolder, F.Cu at (162.8, 95.5)
- added R14: 150, Resistor_SMD:R_0603_1608Metric_Pad0.98x0.95mm_HandSolder, F.Cu at (162.8, 110.2)
- added S1: 219-4MSTR, 219-4MSTR:SOP254P991X385-8N, F.Cu at (148.8, 102.6)
- moved R6 31.9 mm to (162.8, 84.6), turned to 0 degrees
- moved JP1 30.7 mm to (171.4, 119.4)
- moved R9 30.0 mm to (162.8, 91.9)
- moved R5 29.9 mm to (163.6, 119.4)
- moved U2 28.2 mm to (170.2, 115.6)
- moved C7 26.2 mm to (157.2, 95.0)
- moved U3 26.0 mm to (157.2, 89.2)
- moved C5 25.8 mm to (146.8, 112.8)
- moved C4 25.4 mm to (146.8, 119.9)
- moved Y1 25.3 mm to (146.3, 116.3)
- moved U5 24.8 mm to (154.9, 114.6)
- moved C6 21.9 mm to (156.2, 107.7)
- moved R7 21.4 mm to (155.8, 83.6), turned to 0 degrees
- moved C3 21.1 mm to (163.8, 116.1)
- moved R2 20.4 mm to (159.5, 104.6)
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Connections:
- J4 pad 1: unconnected-(J4-Pad1) -> VCC
- J4 pad 10: unconnected-(J4-Pad10) -> /DO_4
- J4 pad 11: unconnected-(J4-Pad11) -> /CAN_H
- J4 pad 12: unconnected-(J4-Pad12) -> /CAN_L
- J4 pad 2: unconnected-(J4-Pad2) -> VCC
- J4 pad 3: unconnected-(J4-Pad3) -> VCC
- J4 pad 4: unconnected-(J4-Pad4) -> GND
- J4 pad 5: unconnected-(J4-Pad5) -> GND
- J4 pad 6: unconnected-(J4-Pad6) -> GND
- J4 pad 7: unconnected-(J4-Pad7) -> /DO_1
- J4 pad 8: unconnected-(J4-Pad8) -> /DO_2
- J4 pad 9: unconnected-(J4-Pad9) -> /DO_3
Other:
- board size 64.3 x 40.6 mm -> 48 x 38.1 mm
- board text added: "2/23/2023"
- board text added: "JHB - CAN 12V DO Board"
- board text removed: "2/17/2023"
- board text removed: "JHB - CAN Relay Board"

Commit message: V1 Schematic and Placement Design complete
Parts:
- added H1: MountingHole, MountingHole:MountingHole_2.2mm_M2_ISO14580, F.Cu at (140.7, 85.1)
- added H2: MountingHole, MountingHole:MountingHole_2.2mm_M2_ISO14580, F.Cu at (140.7, 118.6)
- added R15: ?, Resistor_SMD:R_0603_1608Metric_Pad0.98x0.95mm_HandSolder, F.Cu at (156.2, 99.1)
- added R16: ?, Resistor_SMD:R_0603_1608Metric_Pad0.98x0.95mm_HandSolder, F.Cu at (156.2, 100.8)
- added R17: ?, Resistor_SMD:R_0603_1608Metric_Pad0.98x0.95mm_HandSolder, F.Cu at (156.2, 102.6)
- added R18: ?, Resistor_SMD:R_0603_1608Metric_Pad0.98x0.95mm_HandSolder, F.Cu at (156.2, 104.4)
- added R19: ?, Resistor_SMD:R_0603_1608Metric_Pad0.98x0.95mm_HandSolder, F.Cu at (159.5, 102.6)
- moved D2 7.37 mm to (162.8, 93.7)
- moved D3 7.37 mm to (162.8, 101.1)
- moved R12 7.37 mm to (162.8, 95.5)
- moved R13 7.37 mm to (162.8, 102.9)
- moved R8 7.37 mm to (162.8, 91.9)
- moved R9 7.37 mm to (162.8, 99.3)
- moved U6 7.37 mm to (169.2, 94.2)
- moved U7 7.37 mm to (169.2, 101.6)
- moved R2 3.64 mm to (156.2, 106.2)
- moved R3 2.97 mm to (162.8, 111.8)
- moved C3 1.37 mm to (164.3, 114.8)
- moved C4 0.64 mm to (146.2, 119.9)
- moved C5 0.64 mm to (146.2, 112.8)
- moved Y1 0.64 mm to (145.7, 116.3)
- moved C1 0.57 mm to (145.3, 94.0)
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Connections:
- J3 pad 2: /UART_RX -> unconnected-(J3-Pad2)
- J4 pad 1: VCC -> /CAN_H
- J4 pad 10: /DO_4 -> GND
- J4 pad 11: /CAN_H -> GND
- J4 pad 12: /CAN_L -> GND
- J4 pad 2: VCC -> /CAN_L
- J4 pad 3: VCC -> /DO_4
- J4 pad 4: GND -> /DO_3
- J4 pad 5: GND -> /DO_2
- J4 pad 6: GND -> /DO_1
- J4 pad 7: /DO_1 -> VCC
- J4 pad 8: /DO_2 -> VCC
- J4 pad 9: /DO_3 -> VCC
- S1 pad 1: unconnected-(S1-Pad1) -> +5V
- S1 pad 2: unconnected-(S1-Pad2) -> +5V
- S1 pad 3: unconnected-(S1-Pad3) -> +5V
- S1 pad 4: unconnected-(S1-Pad4) -> +5V
- S1 pad 5: unconnected-(S1-Pad5) -> Net-(R18-Pad2)
- S1 pad 6: unconnected-(S1-Pad6) -> Net-(R17-Pad2)
- S1 pad 7: unconnected-(S1-Pad7) -> Net-(R16-Pad2)
- S1 pad 8: unconnected-(S1-Pad8) -> Net-(R15-Pad2)
- U3 pad 5: /OUT_4 -> /DIP
- U3 pad 6: /UART_RX -> /OUT_4
Routing:
- net +5V: track 0.00 -> 23.7 mm
- net /CAN_H: track 0.00 -> 21.4 mm
- net /CAN_L: track 0.00 -> 19.3 mm
- net Net-(R2-Pad1): track 0.00 -> 13.1 mm
- net Net-(C5-Pad1): track 0.00 -> 13.1 mm
- net Net-(R3-Pad2): track 0.00 -> 10.1 mm
- net /DIP: track 0.00 -> 6.81 mm
- net Net-(C4-Pad1): track 0.00 -> 5.92 mm
- net Net-(JP1-Pad1): track 0.00 -> 5.60 mm
- net /RESET: track 0.00 -> 4.16 mm
- net Net-(R18-Pad2): track 0.00 -> 3.25 mm
- net Net-(R17-Pad2): track 0.00 -> 2.94 mm
- net Net-(R10-Pad2): track 0.00 -> 2.29 mm
- net Net-(R9-Pad2): track 0.00 -> 2.29 mm
- net Net-(R8-Pad2): track 0.00 -> 2.29 mm
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Other:
- board size 48 x 38.1 mm -> 48.8 x 38.1 mm

Commit message: Added rotary switch
Parts:
- S1: value 219-4MSTR -> RDS-10S-7229-A-SMT; footprint 219-4MSTR:SOP254P991X385-8N -> RDS-10S-7229-A-SMT:SW_RDS-10S-7229-A-SMT
- moved J3 2.52 mm to (149.6, 94.2), turned to 90 degrees
- moved S1 0.76 mm to (148.8, 101.9), turned to 90 degrees
Connections:
- S1 pad 1: +5V -> Net-(R15-Pad2)
- S1 pad 2: +5V -> Net-(R16-Pad2)
- S1 pad 4: +5V -> Net-(R17-Pad2)
- S1 pad 8: Net-(R15-Pad2) -> Net-(R18-Pad2)
Changed lines of the file:
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@@
     )
   )
-  (footprint "219-4MSTR:SOP254P991X385-8N" (layer "F.Cu")
-    (at 148.844 102.616)
-    (descr "219-4MSTR")
-    (tags "Switch")
-    (property "Arrow Part Number" "219-4MSTR")
-    (property "Arrow Price/Stock" "https://www.arrow.com/en/products/219-4mstr/cts")
-    (property "Description" "DIP Switches / SIP Switches SPST 4 switch sections")
-    (property "Digi-Key Link" "https://www.digikey.com/en/products/detail/cts-electrocomponents/219-4MSTR/480303")
-    (property "Digi-Key PN" "CT3117CT-ND")
-    (property "Height" "3.85")
-    (property "Manufacturer PN" "219-4MSTR")
-    (property "Manufacturer_Name" "CTS")
-    (property "Manufacturer_Part_Number" "219-4MSTR")
-    (property "Mouser Part Number" "774-2194MSTR")
-    (property "Mouser Price/Stock" "https://www.mouser.co.uk/ProductDetail/CTS-Electronic-Components/219-4MSTR?qs=qNzHFtQhdJ9B7GDGaS2NPg%3D%3D")
-    (property "Price" "0.91")
-    (property "Sheetfile" "CAN-Digital-Output-12V.kicad_sch")
-    (property "Sheetname" "")
-    (attr smd)
-    (fp_text reference "S1" (at 0 0) (layer "F.SilkS")
-      (effects (font (size 1.27 1.27) (thickness 0.254)))
-    )
-    (fp_text value "219-4MSTR" (at 0 0) (layer "F.SilkS") hide
-      (effects (font (size 1.27 1.27) (thickness 0.254)))
-    )
-    (fp_text user "${REFERENCE}" (at 0 0) (layer "F.Fab")
-      (effects (font (size 1.27 1.27) (thickness 0.254)))
-    )
-    (fp_line (start 3 -5.815) (end 3 5.815) (layer "F.SilkS") (width 0.2))
-    (fp_line (start -3 -5.815) (end 3 -5.815) (layer "F.SilkS") (width 0.2))
-    (fp_line (start -5.4 -4.56) (end -3.35 -4.56) (layer "F.SilkS") (width 0.2))
-    (fp_line (start 3 5.815) (end -3 5.815) (layer "F.SilkS") (width 0.2))
-    (fp_line (start -3 5.815) (end -3 -5.815) (layer "F.SilkS") (width 0.2))
-    (fp_line (start 5.65 -6.215) (end 5.65 6.215) (layer "F.CrtYd") (width 0.05))
-    (fp_line (start 5.65 6.215) (end -5.65 6.215) (layer "F.CrtYd") (width 0.05))
-    (fp_line (start -5.65 6.215) (end -5.65 -6.215) (layer "F.CrtYd") (width 0.05))
-    (fp_line (start -5.65 -6.215) (end 5.65 -6.215) (layer "F.CrtYd") (width 0.05))
-    (fp_line (start -3.35 5.815) (end -3.35 -5.815) (layer "F.Fab") (width 0.1))
-    (fp_line (start -3.35 -3.275) (end -0.81 -5.815) (layer "F.Fab") (width 0.1))
-    (fp_line (start 3.35 -5.815) (end 3.35 5.815) (layer "F.Fab") (width 0.1))
-    (fp_line (start 3.35 5.815) (end -3.35 5.815) (layer "F.Fab") (width 0.1))
-    (fp_line (start -3.35 -5.815) (end 3.35 -5.815) (layer "F.Fab") (width 0.1))
-    (pad "1" smd rect (at -4.375 -3.81 90) (size 0.8 2.05) (layers "F.Cu" "F.Paste" "F.Mask")
-      (net 9 "+5V") (pinfunction "1") (pintype "passive"))
-    (pad "2" smd rect (at -4.375 -1.27 90) (size 0.8 2.05) (layers "F.Cu" "F.Paste" "F.Mask")
-      (net 9 "+5V") (pinfunction "2") (pintype "passive"))
-    (pad "3" smd rect (at -4.375 1.27 90) (size 0.8 2.05) (layers "F.Cu" "F.Paste" "F.Mask")
-      (net 9 "+5V") (pinfunction "3") (pintype "passive"))
-    (pad "4" smd rect (at -4.375 3.81 90) (size 0.8 2.05) (layers "F.Cu" "F.Paste" "F.Mask")
-      (net 9 "+5V") (pinfunction "4") (pintype "passive"))
-    (pad "5" smd rect (at 4.375 3.81 90) (size 0.8 2.05) (layers "F.Cu" "F.Paste" "F.Mask")
-      (net 40 "Net-(R18-Pad2)") (pinfunction "5") (pintype "passive"))
-    (pad "6" smd rect (at 4.375 1.27 90) (size 0.8 2.05) (layers "F.Cu" "F.Paste" "F.Mask")
-      (net 39 "Net-(R17-Pad2)") (pinfunction "6") (pintype "passive"))
-    (pad "7" smd rect (at 4.375 -1.27 90) (size 0.8 2.05) (layers "F.Cu" "F.Paste" "F.Mask")
-      (net 38 "Net-(R16-Pad2)") (pinfunction "7") (pintype "passive"))
-    (pad "8" smd rect (at 4.375 -3.81 90) (size 0.8 2.05) (layers "F.Cu" "F.Paste" "F.Mask")
-      (net 37 "Net-(R15-Pad2)") (pinfunction "8") (pintype "passive"))
-    (model "${KIPRJMOD}/Custom Components/219-4MSTR/219-4MSTR.stp"
-      (offset (xyz 0 0 0))
-      (scale (xyz 1 1 1))
-      (rotate (xyz 0 0 0))
+  (footprint "RDS-10S-7229-A-SMT:SW_RDS-10S-7229-A-SMT" (layer "F.Cu")
+    (at 148.844 101.854 90)
+    (property "MANUFACTURER" "CUI Devices")
+    (property "MAXIMUM_PACKAGE_HEIGHT" "3 mm")
+    (property "PARTREV" "1.0")
+    (property "STANDARD" "Manufacturer Recommendations")
+    (property "Sheetfile" "CAN-Digital-Output-12V.kicad_sch")
+    (property "Sheetname" "")
+    (attr smd)
+    (fp_text reference "S1" (at -0.635 -4.445 90) (layer "F.SilkS")
+      (effects (font (size 1 1) (thickness 0.15)))
+    )
+    (fp_text value "RDS-10S-7229-A-SMT" (at 9.525 4.445 90) (layer "F.Fab")
+      (effects (font (size 1 1) (thickness 0.15)))
+    )
+    (fp_line (start 3.6 3.6) (end -3.6 3.6) (layer "F.SilkS") (width 0.127))
+    (fp_line (start -3.6 -3.6) (end 3.6 -3.6) (layer "F.SilkS") (width 0.127))
+    (fp_circle (center 5.927 -0.1) (end 6.027 -0.1) (layer "F.SilkS") (width 0.2) (fill none))
+    (fp_line (start 5.65 -3.85) (end 5.65 3.85) (layer "F.CrtYd") (width 0.05))
+    (fp_line (start 5.65 3.85) (end -5.65 3.85) (layer "F.CrtYd") (width 0.05))
+    (fp_line (start -5.65 3.85) (end -5.65 -3.85) (layer "F.CrtYd") (width 0.05))
+    (fp_line (start -5.65 -3.85) (end 5.65 -3.85) (layer "F.CrtYd") (width 0.05))
+    (fp_line (start -3.6 3.6) (end -3.6 -3.6) (layer "F.Fab") (width 0.127))
+    (fp_line (start -3.6 -3.6) (end 3.6 -3.6) (layer "F.Fab") (width 0.127))
+    (fp_line (start 3.6 -3.6) (end 3.6 3.6) (layer "F.Fab") (width 0.127))
+    (fp_line (start 3.6 3.6) (end -3.6 3.6) (layer "F.Fab") (width 0.127))
+    (fp_circle (center 5.927 -0.1) (end 6.027 -0.1) (layer "F.Fab") (width 0.2) (fill none))
+    (pad "1" smd rect (at 4.4 0 90) (size 2 0.9) (layers "F.Cu" "F.Paste" "F.Mask")
+      (net 37 "Net-(R15-Pad2)") (pinfunction "1") (pintype "passive"))
+    (pad "2" smd rect (at 4.4 -2.54 90) (size 2 0.9) (layers "F.Cu" "F.Paste" "F.Mask")
+      (net 38 "Net-(R16-Pad2)") (pinfunction "2") (pintype "passive"))
+    (pad "4" smd rect (at -4.4 -2.54 90) (size 2 0.9) (layers "F.Cu" "F.Paste" "F.Mask")
+      (net 39 "Net-(R17-Pad2)") (pinfunction "4") (pintype "passive"))
+    (pad "8" smd rect (at -4.4 0 90) (size 2 0.9) (layers "F.Cu" "F.Paste" "F.Mask")
+      (net 40 "Net-(R18-Pad2)") (pinfunction "8") (pintype "passive"))
+    (pad "C1" smd rect (at -4.4 2.54 90) (size 2 0.9) (layers "F.Cu" "F.Paste" "F.Mask")
+      (net 9 "+5V") (pinfunction "C") (pintype "passive"))
+    (pad "C2" smd rect (at 4.4 2.54 90) (size 2 0.9) (layers "F.Cu" "F.Paste" "F.Mask")
+      (net 9 "+5V") (pinfunction "C") (pintype "passive"))
+    (model "${KIPRJMOD}/Custom Components/RDS-10S-7229-A-SMT/CUI_DEVICES_RDS-10S-7229-A-SMT.step"
+      (offset (xyz -4.8 6.35 -4.4))
+      (scale (xyz 1 1 1))
+      (rotate (xyz -90 0 0))
     )
   )
@@
   )
   (footprint "Connector_PinHeader_1.27mm:PinHeader_1x03_P1.27mm_Vertical" (layer "F.Cu")
-    (at 151.384 92.456)
+    (at 149.601 94.234 90)
     (descr "Through hole straight pin header, 1x03, 1.27mm pitch, single row")
     (tags "Through hole pin header THT 1x03 1.27mm single row")
@@
     (property "Sheetname" "")
     (attr through_hole)
-    (fp_text reference "J3" (at 1.27 -1.27 90) (layer "F.SilkS") hide
-      (effects (font (size 1 1) (thickness 0.15)))
-    )
-    (fp_text value "UART Header" (at 0 4.235) (layer "F.Fab")
-      (effects (font (size 1 1) (thickness 0.15)))
-    )
-    (fp_text user "${REFERENCE}" (at 0 1.27 90) (layer "F.Fab")
+    (fp_text reference "J3" (at 1.27 -1.27) (layer "F.SilkS") hide
+      (effects (font (size 1 1) (thickness 0.15)))
+    )
+    (fp_text value "UART Header" (at 0 4.235 90) (layer "F.Fab")
+      (effects (font (size 1 1) (thickness 0.15)))
+    )
+    (fp_text user "${REFERENCE}" (at 0 1.27) (layer "F.Fab")
       (effects (font (size 1 1) (thickness 0.15)))
     )
@@
     (fp_line (start -1.05 -0.11) (end -0.525 -0.635) (layer "F.Fab") (width 0.1))
     (fp_line (start 1.05 -0.635) (end 1.05 3.175) (layer "F.Fab") (width 0.1))
-    (pad "1" thru_hole rect (at 0 0) (size 1 1) (drill 0.65) (layers *.Cu *.Mask)
+    (pad "1" thru_hole rect (at 0 0 90) (size 1 1) (drill 0.65) (layers *.Cu *.Mask)
       (net 8 "GND") (pinfunction "Pin_1") (pintype "passive"))
-    (pad "2" thru_hole oval (at 0 1.27) (size 1 1) (drill 0.65) (layers *.Cu *.Mask)
+    (pad "2" thru_hole oval (at 0 1.27 90) (size 1 1) (drill 0.65) (layers *.Cu *.Mask)
       (net 5 "unconnected-(J3-Pad2)") (pinfunction "Pin_2") (pintype "passive"))
-    (pad "3" thru_hole oval (at 0 2.54) (size 1 1) (drill 0.65) (layers *.Cu *.Mask)
+    (pad "3" thru_hole oval (at 0 2.54 90) (size 1 1) (drill 0.65) (layers *.Cu *.Mask)
       (net 10 "/UART_TX") (pinfunction "Pin_3") (pintype "passive"))
     (model "${KICAD6_3DMODEL_DIR}/Connector_PinHeader_1.27mm.3dshapes/PinHeader_1x03_P1.27mm_Vertical.wrl"
@@
   (gr_line (start 187.198 120.904) (end 138.43 120.904) (layer "Edge.Cuts") (width 0.1))
   (gr_line (start 138.43 82.804) (end 138.43 87.376) (layer "Edge.Cuts") (width 0.1))
+  (gr_line (start 148.844 101.854) (end 136.652 101.854) (layer "B.Fab") (width 0.1))
   (gr_rect (start 187.198 120.904) (end 142.748 82.804) (layer "B.Fab") (width 0.1) (fill none))
   (gr_rect (start 138.43 82.804) (end 142.748 87.376) (layer "B.Fab") (width 0.2) (fill none))
@@
       (effects (font (size 1 1) (thickness 0.15)))
     )
+    (format (units 3) (units_format 1) (precision 4))
+    (style (thickness 0.1) (arrow_length 1.27) (text_position_mode 0) (extension_height 0.58642) (extension_offset 0.5) keep_text_aligned)
+  )
+  (dimension (type aligned) (layer "B.Fab")
+    (pts (xy 137.16 101.854) (xy 137.160001 120.904))
+    (height 5.588)
+    (gr_text "19.0500 mm" (at 130.422 111.379 90) (layer "B.Fab")
+      (effects (font (size 1 1) (thickness 0.15)))
+    )

Commit message: Sent to Fab
Parts:
- removed J1: UPDI Header, Connector_PinHeader_1.27mm:PinHeader_1x02_P1.27mm_Vertical
- J3: value UART Header -> UPDI Header
- moved R7 11.5 mm to (154.2, 95.0)
- moved R1 3.88 mm to (156.2, 104.1), turned to 0 degrees
- moved C2 2.79 mm to (148.1, 84.3)
- moved R18 1.78 mm to (156.2, 102.6)
- moved R15 1.52 mm to (156.2, 97.5)
- moved R16 1.52 mm to (156.2, 99.3)
- moved R17 1.52 mm to (156.2, 101.1)
- moved J3 1.05 mm to (148.6, 94.5)
- moved R19 1.02 mm to (159.5, 101.6)
- moved C4 0.92 mm to (146.1, 119.0)
- moved Y1 0.92 mm to (145.5, 115.4)
- moved C5 0.92 mm to (146.1, 111.9)
- moved C7 0.76 mm to (158.0, 95.0)
Connections:
- J3 pad 2: unconnected-(J3-Pad2) -> /UART_TX
- J3 pad 3: /UART_TX -> Net-(J3-Pad3)
- R7 pad 1: Net-(J1-Pad1) -> Net-(J3-Pad3)
Routing:
- net VCC: track 0.00 -> 63.0 mm, vias 0 -> 2
- net +5V: track 23.7 -> 76.2 mm, vias 0 -> 5
- net /INT: track 0.00 -> 38.1 mm, vias 0 -> 2
- net /CS: track 0.00 -> 36.4 mm, vias 0 -> 3
- net /MOSI: track 0.00 -> 33.5 mm, vias 0 -> 2
- net /SCK: track 0.00 -> 31.5 mm, vias 0 -> 2
- net Net-(U2-Pad1): track 0.00 -> 30.7 mm, vias 0 -> 2
- net /MISO: track 0.00 -> 30.1 mm, vias 0 -> 2
- net Net-(U2-Pad4): track 0.00 -> 29.7 mm, vias 0 -> 2
- net /OUT_4: track 1.79 -> 27.4 mm, vias 0 -> 2
- net /DIP: track 6.81 -> 27.4 mm, vias 0 -> 2
- net /UART_TX: track 0.00 -> 19.8 mm
- net /DO_1: track 0.00 -> 15.0 mm
- net /DO_4: track 0.00 -> 13.0 mm
- net /OUT_3: track 1.79 -> 13.1 mm, vias 0 -> 2
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Other:
- board text added: "2/26/2023"
- board text removed: "2/23/2023"
